Commit message: Verbindung des RobotiQ Grippers an UR3
Weiter bestehendes Problem:
Found a contact between 'robotiq_85_right_inner_knuckle_link' (type 'Robot link') and 'robotiq_85_right_finger_tip_link' (type 'Robot link'), which constitutes a collision. Contact information is not stored.

File: ur3_robotiq85_gripper.urdf.xacro (robot description, xacro)
@@ -28,9 +28,17 @@
     <origin xyz="0.0 0.0 0.0" rpy="0.0 0.0 0.0" />
   </joint>
-  <joint name="tool0" type="fixed">
+  <!-- Robotiq Coupler Joint an tool0-Link -->
+  <joint name="robotiq_coupler_joint" type="fixed">
+    <origin xyz="0 0 0.04" rpy="0 0 ${-pi/2.0}" />
+    <parent link="tool0"/>
+    <child link="robotiq_coupler"/>
+  </joint>
+  <!-- oder alternativ dazu
+  <joint name="ee_link" type="fixed">
     <parent link="wrist_3_link" />
     <child link = "robotiq_coupler" />
     <origin xyz="0.0 0.0 0.0" rpy="0.0 0.0 0.0" />
   </joint>
+  -->
   <!-- Robotiq Coupler -->
   <!--  + Height added by the coupler: 8mm -->
@@ -49,5 +57,5 @@
     </collision>
     <inertial>
-      <origin xyz="2.073e-05   1.45286e-03  -1.1049e-03" rpy="0 0 0" />
+      <origin xyz="0 0 0" rpy="0 0 0" />
       <mass value="0.168" />
       <inertia ixx="6.69695624e-05" ixy="5.21511788e-09" ixz="-2.74383009e-08"
@@ -55,9 +63,4 @@
     </inertial>
   </link>
-  <joint name="robotiq_coupler_joint" type="fixed">
-    <origin xyz="0 0 0.004" rpy="0 0 ${-pi/2.0}" />
-    <parent link="tool0"/>
-    <child link="robotiq_coupler"/>
-  </joint>
   <gazebo reference="robotiq_coupler">
     <mu1>0.9</mu1>
@@ -67,5 +70,5 @@
   <!-- Attach the robotiq 85 gripper -->
   <xacro:robotiq_85_gripper prefix="" parent="robotiq_coupler" >
-    <origin xyz="0 0 0.004" rpy="0 ${-pi/2} ${pi}"/>
+    <origin xyz="0 0 0.00" rpy="0 ${-pi/2} ${pi}"/>
   </xacro:robotiq_85_gripper>
 </robot>
